Commit message: blah blah

File: install/arduinobot_description/share/arduinobot_description/urdf/arduinobot.urdf.xacro (robot description, xacro)
@@ -1,8 +1,16 @@
-<?xml version="1.0" encoding="UTF-8"?>
+<?xml version="1.0"?>
 <robot xmlns:xacro="http://www.ros.org/wiki/xacro" name="arduinobot">
-    <!--xacro lets you define variables -->
-    <xacro:property name="PI" value="3.14159"></xacro:property>
-    <xacro:property name="effort" value="30.0"></xacro:property>
-    <xacro:property name="velocity" value="10.0"></xacro:property>
+    <!-- Start GZ or Ignition depending on ROS 2 Version -->
+    <xacro:arg name="is_ignition" default="true"/>
+    <!-- Load Simulated or Real Hardware Interfaces -->
+    <xacro:arg name="is_sim" default="true"/>
+    <!-- Include Gazebo Parameters -->
+    <xacro:include filename="$(find arduinobot_description)/urdf/arduinobot_gazebo.xacro" />
+    <!-- Include ros2_control Plugins -->
+    <xacro:include filename="$(find arduinobot_description)/urdf/arduinobot_ros2_control.xacro" />
+    <!-- Useful XACRO Variables (Properties) -->
+    <xacro:property name="PI" value="3.14159265359" />
+    <xacro:property name="effort" value="30.0" />
+    <xacro:property name="velocity" value="10.0" />
     <!-- Useful Macros -->
     <xacro:macro name="default_inertial" params="mass">
@@ -15,62 +23,40 @@
         </inertial>
     </xacro:macro>
-    <link name="world"> <!--Link is the RIGID body of the robot, a single component, viual prperties and POSE-->
-    </link>
+    <!-- Links -->
+    <link name="world"/>
     <link name="base_link">
-        <xacro:default_inertial mass="1.0"></xacro:default_inertial>
-        <!-- The visual appearnce of the robot; shape, size position and materials etc-->
+        <xacro:default_inertial mass="1.0"/>
         <visual>
-            <!-- Specified the position and orientation (pose); xyz = 0 0 0 means that it is located exactly in the middle; rpy = 0 0 0 means there is also no roation along the 3 axises-->
             <origin rpy="0 0 0" xyz="-0.5 -0.5 0"/>
-            <!-- specified the shape of the link; in our example we have external files to describe the actual link-->
             <geometry>
-                <mesh filename="package://arduinobot_description/meshes/basement.STL" scale= "0.01 0.01 0.01"/>
+                <mesh filename="package://arduinobot_description/meshes/basement.STL" scale="0.01 0.01 0.01"/>
             </geometry>
         </visual>
         <collision>
-        <origin rpy="0 0 0" xyz="-0.5 -0.5 0"/>
-            <!-- specified the shape of the link; in our example we have external files to describe the actual link-->
+            <origin rpy="0 0 0" xyz="-0.5 -0.5 0"/>
             <geometry>
-                <mesh filename="package://arduinobot_description/meshes/basement.STL" scale= "0.01 0.01 0.01"/>
+                <mesh filename="package://arduinobot_description/meshes/basement.STL" scale="0.01 0.01 0.01"/>
             </geometry>
         </collision>
     </link>
-    <!-- Joint tags define the connection of links and how they move relative to each other-->
-    <!-- Also described the type of link, in this case fixed which means that no relative motion between the link; but you can also have revolute type which means rotational motion about a single axis-->
-    <!-- Fixed is a static connection, it can not move with respect to any other links it may be jointed with-->
-    <joint name="virtual_joint" type="fixed">
-        <parent link="world"></parent>
-        <child link="base_link"></child>
-        <origin rpy="0 0 0" xyz="0 0 0"></origin>
-    </joint>
     <link name="base_plate">
-        <xacro:default_inertial mass="0.1"></xacro:default_inertial>
+        <xacro:default_inertial mass="0.1"/>
         <visual>
-            <origin rpy="0 0 0" xyz="-0.39 -0.39 -0.56"></origin>
-                <geometry>
-                    <mesh filename="package://arduinobot_description/meshes/base_plate.STL" scale="0.01 0.01 0.01"></mesh>
-                </geometry>
+            <origin rpy="0 0 0" xyz="-0.39 -0.39 -0.56"/>
+            <geometry>
+                <mesh filename="package://arduinobot_description/meshes/base_plate.STL" scale="0.01 0.01 0.01"/>
+            </geometry>
         </visual>
         <collision>
-        <origin rpy="0 0 0" xyz="-0.39 -0.39 -0.56"></origin>
-                <geometry>
-                    <mesh filename="package://arduinobot_description/meshes/base_plate.STL" scale="0.01 0.01 0.01"></mesh>
-                </geometry>
+            <origin rpy="0 0 0" xyz="-0.39 -0.39 -0.56"/>
+            <geometry>
+                <mesh filename="package://arduinobot_description/meshes/base_plate.STL" scale="0.01 0.01 0.01"/>
+            </geometry>
         </collision>
     </link>
-    <!-- Revolute joint means the baseplate can rotate with respect to its parent; in the axis tag we set that they can rotate on the z axis-->
-    <joint name="joint_1" type="revolute">
-        <parent link="base_link"></parent>
-        <child link="base_plate"></child>
-        <axis xyz="0 0 1"></axis>
-        <!-- Transformation matrix that connects the base link with the base plate-->
-        <origin rpy="0 0 0" xyz="0 0 0.307"></origin>
-        <!-- Limits on the roation -->
-        <limit lower="-${PI/2}" upper="${PI/2}" effort="${effort}" velocity="${velocity}"></limit>
-    </joint>
     <link name="forward_drive_arm">
-        <xacro:default_inertial mass="0.1"></xacro:default_inertial>
+        <xacro:default_inertial mass="0.1"/>
         <visual>
-            <origin rpy="0 -${PI/2} ${PI/2}" xyz="0.19 0.06 -0.08"/>
+            <origin rpy=" 0 -${PI / 2} ${PI / 2}" xyz="0.19 0.06 -0.08"/>
             <geometry>
                 <mesh filename="package://arduinobot_description/meshes/forward_drive_arm.STL" scale="0.01 0.01 0.01"/>
@@ -78,5 +64,5 @@
         </visual>
         <collision>
-        <origin rpy="0 -${PI/2} ${PI/2}" xyz="0.19 0.06 -0.08"/>
+            <origin rpy=" 0 -${PI / 2} ${PI / 2}" xyz="0.19 0.06 -0.08"/>
             <geometry>
                 <mesh filename="package://arduinobot_description/meshes/forward_drive_arm.STL" scale="0.01 0.01 0.01"/>
@@ -84,15 +70,8 @@
         </collision>
     </link>
-    <joint name="joint_2" type="revolute">
-        <parent link="base_plate"/>
-        <child link="forward_drive_arm"/>
-        <axis xyz="1 0 0"/>
-        <origin rpy="0 0 0" xyz="-0.02 0 0.35"/>
-        <limit lower="-${PI/2}" upper="${PI/2}" effort="${effort}" velocity="${velocity}"/>
-    </joint>
     <link name="horizontal_arm">
-        <xacro:default_inertial mass="0.1"></xacro:default_inertial>
+        <xacro:default_inertial mass="0.1"/>
         <visual>
-            <origin rpy="${PI/2} 0 ${PI/2}" xyz="-0.03 -0.4 -0.06"/>
+            <origin rpy="${PI / 2} 0 ${PI / 2}" xyz="-0.03 -0.4 -0.06"/>
             <geometry>
                 <mesh filename="package://arduinobot_description/meshes/horizontal_arm.STL" scale="0.01 0.01 0.01"/>
@@ -100,5 +79,5 @@
         </visual>
         <collision>
-        <origin rpy="${PI/2} 0 ${PI/2}" xyz="-0.03 -0.4 -0.06"/>
+            <origin rpy="${PI / 2} 0 ${PI / 2}" xyz="-0.03 -0.4 -0.06"/>
             <geometry>
                 <mesh filename="package://arduinobot_description/meshes/horizontal_arm.STL" scale="0.01 0.01 0.01"/>
@@ -106,11 +85,4 @@
         </collision>
     </link>
-    <joint name="joint_3" type="revolute">
-        <parent link="forward_drive_arm"/>
-        <child link="horizontal_arm"/>
-        <axis xyz="1 0 0"/>
-        <origin rpy="0 0 0" xyz="0 0 0.8"/>
-        <limit lower="-${PI/2}" upper="${PI/2}" effort="${effort}" velocity="${velocity}"/>
-    </joint>
     <link name="claw_support">
         <xacro:default_inertial mass="0.05"/>
@@ -128,9 +100,4 @@
         </collision>
     </link>
-    <joint name="horizontal_arm_to_claw_support" type="fixed">
-        <parent link="horizontal_arm"/>
-        <child link="claw_support"/>
-        <origin xyz="0 0.82 0" rpy="0 0 0"/>
-    </joint>
     <link name="gripper_right">
         <xacro:default_inertial mass="0.01"/>
@@ -148,5 +115,5 @@
         </collision>
     </link>
-      <link name="gripper_left">
+    <link name="gripper_left">
         <xacro:default_inertial mass="0.01"/>
         <visual>
@@ -163,5 +130,40 @@
         </collision>
     </link>
-   <joint name ="joint_4" type="revolute">
+    <!-- Joints -->
+    <joint name="virtual_joint" type="fixed">
+        <parent link="world"/>
+        <child link="base_link"/>
+        <origin xyz="0 0 0" rpy="0 0 0"/>
+    </joint>
+    <joint name ="joint_1" type="revolute">
+        <parent link="base_link"/>
+        <child link = "base_plate"/>
+        <origin xyz="0 0 0.307"/>
+        <axis xyz="0 0 1"/>
+        <limit lower="-${PI / 2}" upper="${PI / 2}"
+               effort="${effort}" velocity="${velocity}"/>
+    </joint>
+    <joint name ="joint_2" type="revolute">
+        <parent link="base_plate"/>
+        <child link = "forward_drive_arm"/>
+        <origin xyz="-0.02 0 0.35"/>
+        <axis xyz="1 0 0"/>
+        <limit lower="-${PI / 2}" upper="${PI / 2}"
+                effort="${effort}" velocity="${velocity}"/>
+    </joint>
+    <joint name ="joint_3" type="revolute">
+        <parent link="forward_drive_arm"/>
+        <child link = "horizontal_arm"/>
+        <origin xyz="0 0 0.8"/>
+        <axis xyz="1 0 0"/>
+        <limit lower="-${PI / 2}" upper="${PI / 2}"
+               effort="${effort}" velocity="${velocity}"/>
+    </joint>
+    <joint name ="horizontal_arm_to_claw_support" type="fixed">
+        <parent link="horizontal_arm"/>
+        <child link = "claw_support"/>
+        <origin xyz="0 0.82 0"/>
+    </joint>
+    <joint name ="joint_4" type="revolute">
         <parent link="claw_support"/>
         <child link = "gripper_right"/>
@@ -180,26 +182,3 @@
         <mimic joint="joint_4" multiplier="-1"/>
     </joint>
-    <link name="rgb_camera">
-        <!-- The visual appearnce of the robot; shape, size position and materials etc-->
-        <visual>
-            <!-- Specified the position and orientation (pose); xyz = 0 0 0 means that it is located exactly in the middle; rpy = 0 0 0 means there is also no roation along the 3 axises-->
-            <origin rpy="1.57 3.14 1.57" xyz="0 0.12 0.2"/>
-            <!-- specified the shape of the link; in our example we have external files to describe the actual link-->
-            <geometry>
-                <mesh filename="package://arduinobot_description/meshes/pi_camera.STL" scale= "0.01 0.01 0.01"/>
-            </geometry>
-        </visual>
-        <collision>
-        <origin rpy="1.57 3.14 1.57" xyz="0 0.12 0.2"/>
-            <!-- specified the shape of the link; in our example we have external files to describe the actual link-->
-            <geometry>
-                <mesh filename="package://arduinobot_description/meshes/pi_camera.STL" scale= "0.01 0.01 0.01"/>
-            </geometry>
-        </collision>
-    </link>
-    <joint name ="joint_6" type="fixed">
-        <parent link="base_link"/>
-        <child link = "rgb_camera"/>
-        <origin rpy="0 -0.5 1.57" xyz="0 0.45 0.2"/>
-    </joint>
 </robot>
